File: flowsense_charger.kicad_sch (KiCad schematic)
At the start: 34 parts, among them J1 SOLAR, J2 LOAD, J3 Conn_01x02_Pin, J4 Conn_02x20_Odd_Even, J5 USB_A, SW1 SW_Push, U1 BQ25185, U2 TPS61230DRC

Commit message: Scheme: Fixes capacitor issue on PIN1 SYS of U1. Adds decoupler 1uF on PIN2 BAT of U1. Clarifies text
Parts:
- removed D3: LED, LED_SMD:LED_1206_3216Metric_Pad1.42x1.75mm_HandSolder, symbol Device:LED
- removed J4: Conn_02x20_Odd_Even, Connector_PinHeader_2.54mm:PinHeader_2x20_P2.54mm_Vertical, symbol Connector_Generic:Conn_02x20_Odd_Even
- removed JP3_ISET_1A1, JP4_ISET_500mA1: SolderJumper_2_Open, Jumper:SolderJumper-2_P1.3mm_Open_Pad1.0x1.5mm, symbol Jumper:SolderJumper_2_Open
- removed R10: 470, Resistor_SMD:R_1206_3216Metric, symbol Device:R
- removed R4: 600 ohm, Resistor_SMD:R_1206_3216Metric, symbol Device:R
- added C6: 1uF, symbol Device:C
- added J4: LOAD, TerminalBlock_Phoenix:TerminalBlock_Phoenix_MPT-0,5-2-2.54_1x02_P2.54mm_Horizontal, symbol Connector:Conn_01x02_Socket
- added J6: Conn_01x02_Pin, TerminalBlock_Phoenix:TerminalBlock_Phoenix_MPT-0,5-2-2.54_1x02_P2.54mm_Horizontal, symbol Connector:Conn_01x02_Pin
- added J7: SOLAR, TerminalBlock_Phoenix:TerminalBlock_Phoenix_MPT-0,5-2-2.54_1x02_P2.54mm_Horizontal, symbol Connector:Conn_01x02_Socket
- added JP1: SJ2, Jumper:SolderJumper-2_P1.3mm_Bridged_Pad1.0x1.5mm, symbol Jumper:SolderJumper_2_Bridged
- added R11: 600 ohm, Resistor_SMD:R_1206_3216Metric, symbol Device:R
- C2: value 1uF -> 10uF
- R3: value 300 ohm -> 600 ohm
Connections:
- net +5V: now also J4.2 (Pin_2)
- net +BATT: now also C6.2, J6.1 (Pin_1)
- net GND: now also C6.1, J4.1 (Pin_1), J6.2 (Pin_2), J7.1 (Pin_1), JP1.1 (A), R11.2
- net ISET: now also R11.1
- net at C1.1, J1.2 (Pin_2), U1.10 (IN): now also J7.2 (Pin_2)
- net at R3.2: now also JP1.2 (B)
- no-connect marks 33 -> 4
Other:
- note added: "3.7v, one cell, li-po battery (max 4.2V!)- input (IN PIN) current limiting (current from solar panel) 13Kohm for 4.2V chemistery and 1100mA 18Kohm for 4.2V chemistery and 500mA !! Only solder one of the jumpers !! !! Set according to your solar panel current and cell chemistry !!"
- note added: "4.5v from BQ chip Max 3.12A"
- note added: "Absolute maximum ratings -0.3V - 25V Recommended operating conditions: 2.7V-5.5V Operating solar input voltage range: 3.6V-18V"
- note added: "Battery output to positive terminal"
- note added: "Charging current limiting Charge current factor typ: 300 A*Ohm 1A charge (default): Set ISET to 300 Ohm 500mA charge: cut JP1, sets ISET to 600 Ohm !! Set according to your cells charging current capabilities !!"
- note added: "Works for LiFe/LiPo"
- note removed: "4.2V battery - input (IN PIN) current limiting (current from solar panel) Only solder one of the jumpers 13Kohm for 4.2V chemisteries and 1100mA 18Kohm for 4.2V chemistery and 500mA"
- note removed: "4.5v"
- note removed: "Absolute maximum ratings -0.3V - 25V Recommended operating conditions: 2.7-5.5 Operating Vin voltage range: 3.6-18"
- note removed: "Battery output"
- note removed: "Charge current limiting"
- moved on the sheet: C2, DS2, JP1_1100mA_4.2v1, JP2_500mA_4.2v1, R1, R2, R3, R8, TP1, TP2, TP3
