File: flowsense_charger.kicad_sch (KiCad schematic)
At the start: 39 parts, among them J1 SOLAR, J2 LOAD, J3 Conn_01x02_Pin, J4 LOAD, J5 USB_A, J6 Conn_01x02_Pin, J7 SOLAR, J8 Conn_01x02_Pin, J9 Conn_01x02_Pin, SW1 SW_Push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

Commit message: Removes old design file. Updates current file with design that passes DRC.
Parts:
- renumbered JP1_1100mA_4.2v1 to 1100mA_4.2v1, JP2_500mA_4.2v1 to 500mA_4.2v1
Changed lines of the file:
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@@
 		(on_board yes)
 		(dnp no)
-		(property "Reference" "JP1_1100mA_4.2v1"
+		(property "Reference" "1100mA_4.2v1"
 			(at 20.32 52.07 0)
 			(effects
@@
 			(project "flowsense_charger"
 				(path "/06a81c65-da63-44d6-adfc-3d6276b1b4c5"
-					(reference "JP1_1100mA_4.2v1")
+					(reference "1100mA_4.2v1")
 					(unit 1)
 				)
@@
 		(on_board yes)
 		(dnp no)
-		(property "Reference" "JP2_500mA_4.2v1"
+		(property "Reference" "500mA_4.2v1"
 			(at 34.29 72.39 0)
 			(effects
@@
 			(project "flowsense_charger"
 				(path "/06a81c65-da63-44d6-adfc-3d6276b1b4c5"
-					(reference "JP2_500mA_4.2v1")
+					(reference "500mA_4.2v1")
 					(unit 1)
 				)
@@
 		(exclude_from_sim no)
 		(in_bom yes)
-		(on_board yes)
+		(on_board no)
 		(dnp yes)
 		(fields_autoplaced yes)
